Commit message: origin update
changed origin in xacro so the lasers flush against base
also updated urdf file based on updated xacro file

File: urdf/robot.urdf (robot description, URDF)
Before this commit: robot navvis, 6 links, 5 joints
Links:
- added link laser_horiz, mass 0.01; collision sphere radius=0; visual mesh filename=package://velodyne_description/meshes/VLP16_scan.dae
- added link laser_horiz_base_link, mass 0.83; collision cylinder length=0.0717 radius=0.0516; visual mesh filename=package://velodyne_description/meshes/VLP16_base_1.dae
- added link laser_vert_bottom, mass 1e-5; collision box size=0.1 0.1 0.1; visual mesh filename=package://gazebo_plugins/test/multi_robot_scenario/meshes/l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
- added link wheel_center_link; collision cylinder length=0.05 radius=0.15; visual cylinder length=0.05 radius=0.15
- added link wheel_right_link; collision cylinder length=0.05 radius=0.2; visual cylinder length=0.05 radius=0.2
Joints:
- added joint base_link_laser_vert_bottom_joint: type fixed, parent base_link, child laser_vert_bottom, origin xyz=0.3157894464801903 -0.002068548615034871 0.5099999434059285 rpy=3.1354753 -1.3045001 0.0024658, axis 0 0 1
- added joint base_wheel_center_joint: type continuous, parent base_link, child wheel_center_link, origin xyz=0.10 0.0 0.0 rpy=-1.57 0.0 0.0, axis 0 0 1, limit effort=10000 velocity=10000
- added joint base_wheel_right_joint: type continuous, parent base_link, child wheel_right_link, origin xyz=-0.10 -0.4 0.0 rpy=-1.57 0.0 0.0, axis 0 0 1, limit effort=10000 velocity=10000
- added joint laser_horiz_base_mount_joint: type fixed, parent base_link, child laser_horiz_base_link, origin xyz=0.2325416305773505 -0.0001380069427607134 1.920122926231907 rpy=-0.0012068 0.114646 -0.0015308
- added joint laser_horiz_base_scan_joint: type fixed, parent laser_horiz_base_link, child laser_horiz, origin xyz=0 0 0.0377 rpy=0 0 0
- joint base_wheel_left_joint: axis (none) -> 0 0 1; limit (none) -> effort=10000 velocity=10000; origin xyz=-0.10 0.4 0.0 rpy=1.57 0.0 0.0 -> xyz=-0.10 0.4 0.0 rpy=-1.57 0.0 0.0; type fixed -> continuous

File: urdf/robot.xacro (robot description, xacro)
@@ -1,4 +1,7 @@
 <?xml version="1.0"?>
 <robot xmlns:xacro="http://www.ros.org/wiki/xacro" name="navvis">
+    <xacro:include filename="$(find
+    gazebo_plugins)/test/multi_robot_scenario/xacro/laser/hokuyo.xacro" />
+    <xacro:include filename="$(find velodyne_description)/urdf/VLP-16.urdf.xacro" />
     <link name="base_link">
         <visual>
@@ -17,5 +20,4 @@
     <link name="laser_vert_bottom_link">
         <visual>
-        <origin xyz="0.3158 -0.0021 0.5100" rpy="3.1355 -1.3045 0.0025" />
                 <geometry>
                     <box size ="0.062 0.062 0.087" />
@@ -23,5 +25,4 @@
         </visual>
         <collision>
-        <origin xyz="0.3158 -0.0021 0.5100" rpy="3.1355 -1.3045 0.0025" />
                 <geometry>
                     <box size ="0.062 0.062 0.087" />
@@ -37,5 +38,4 @@
     <link name="laser_vert_top_right_link">
         <visual>
-        <origin xyz="0.2978 -0.1450 1.8451" rpy="-1.1760 0.6313 -1.9377" />
                 <geometry>
                     <box size ="0.062 0.062 0.087" />
@@ -43,5 +43,4 @@
         </visual>
         <collision>
-        <origin xyz="0.2978 -0.1450 1.8451" rpy="-1.1760 0.6313 -1.9377" />
                 <geometry>
                     <box size ="0.062 0.062 0.087" />
@@ -56,5 +55,4 @@
     <link name="laser_vert_top_left_link">
         <visual>
-        <origin xyz="0.2997 0.1531 1.8443" rpy="1.1780 0.6198 1.9560" />
                 <geometry>
                     <box size ="0.062 0.062 0.087" />
@@ -62,5 +60,4 @@
         </visual>
         <collision>
-        <origin xyz="0.2997 0.1531 1.8443" rpy="1.1780 0.6198 1.9560" />
                 <geometry>
                     <box size ="0.062 0.062 0.087" />
@@ -75,5 +72,4 @@
     <link name="laser_horiz_link">
         <visual>
-        <origin xyz="0.2325 0.0001 1.9201" rpy="-0.0012 0.1146 -0.0015" />
                 <geometry>
                     <cylinder radius ="0.0652" length="0.072" />
@@ -81,5 +77,4 @@
         </visual>
         <collision>
-        <origin xyz="0.2325 0.0001 1.9201" rpy="-0.0012 0.1146 -0.0015" />
                 <geometry>
                     <cylinder radius ="0.0652" length="0.072" />
@@ -134,9 +129,6 @@
     <xacro:xacro_name side="left" reflect="1" />
     <xacro:xacro_name side="right" reflect="-1" />
-    <xacro:include filename="$(find
-            gazebo_plugins)/test/multi_robot_scenario/xacro/laser/hokuyo.xacro" />
     <xacro:laser name="laser_vert_bottom" parent="base_link" xyz="0.3157894464801903 -0.002068548615034871 0.5099999434059285"
             rpy="3.1354753 -1.3045001 0.0024658" meshes="package://gazebo_plugins/test/multi_robot_scenario/meshes/laser" />
-    <xacro:include filename="$(find velodyne_description)/urdf/VLP-16.urdf.xacro" />
     <xacro:VLP-16 parent="base_link" name="laser_horiz" topic="laser_horiz/packets"
         hz="10" samples="440" gpu="false" >

Commit message: update to robot description and launch
went back and saw not all the meshes were added which is why they weren't appearing
added the laser_vert_top_left|right

the launch file has been updated according to lab 3

File: urdf/robot.urdf (robot description, URDF)
Before this commit: robot navvis, 11 links, 10 joints
Links:
- removed link base_link
- removed link laser_horiz_link
- removed link laser_vert_bottom_link
- removed link laser_vert_top_left_link
- removed link laser_vert_top_right_link
- added link base; collision box size=0.45 0.78 1.98; visual box size=0.45 0.78 1.98
- added link laser_vert_top_left, mass 1e-5; collision box size=0.1 0.1 0.1; visual mesh filename=package://gazebo_plugins/test/multi_robot_scenario/meshes/l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
- added link laser_vert_top_right, mass 1e-5; collision box size=0.1 0.1 0.1; visual mesh filename=package://gazebo_plugins/test/multi_robot_scenario/meshes/l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
Joints:
- removed joint base_laser_horiz_joint
- removed joint base_link_laser_vert_bottom_joint
- joint base_laser_vert_bottom_joint: axis (none) -> 0 0 1; child laser_vert_bottom_link -> laser_vert_bottom; origin xyz=0.3158 -0.0021 0.5100 rpy=3.1355 -1.3045 0.0025 -> xyz=0.3157894464801903 -0.002068548615034871 0.5099999434059285 rpy=3.1354753 -1.3045001 0.0024658; parent base_link -> base
- joint base_laser_vert_top_left_joint: axis (none) -> 0 0 1; child laser_vert_top_left_link -> laser_vert_top_left; parent base_link -> base
- joint base_laser_vert_top_right_joint: axis (none) -> 0 0 1; child laser_vert_top_right_link -> laser_vert_top_right; parent base_link -> base
- joint base_wheel_center_joint: parent base_link -> base
- joint base_wheel_left_joint: parent base_link -> base
- joint base_wheel_right_joint: parent base_link -> base
- joint laser_horiz_base_mount_joint: parent base_link -> base

File: urdf/robot.xacro (robot description, xacro)
@@ -4,5 +4,5 @@
     gazebo_plugins)/test/multi_robot_scenario/xacro/laser/hokuyo.xacro" />
     <xacro:include filename="$(find velodyne_description)/urdf/VLP-16.urdf.xacro" />
-    <link name="base_link">
+    <link name="base">
         <visual>
         <origin xyz="0.0 0.0 0.96" rpy="0.0 0.0 0.0" />
@@ -18,73 +18,4 @@
         </collision>
     </link>
-    <link name="laser_vert_bottom_link">
-        <visual>
-                <geometry>
-                    <box size ="0.062 0.062 0.087" />
-                </geometry>
-        </visual>
-        <collision>
-                <geometry>
-                    <box size ="0.062 0.062 0.087" />
-                </geometry>
-        </collision>
-    </link>
-    <!-- origin of joint is point of refernce where the parent and child link attach !-->
-    <joint name="base_laser_vert_bottom_joint" type="fixed">
-        <parent link="base_link" />
-        <child link="laser_vert_bottom_link" />
-        <origin xyz="0.3158 -0.0021 0.5100" rpy="3.1355 -1.3045 0.0025" />
-    </joint>
-    <link name="laser_vert_top_right_link">
-        <visual>
-                <geometry>
-                    <box size ="0.062 0.062 0.087" />
-                </geometry>
-        </visual>
-        <collision>
-                <geometry>
-                    <box size ="0.062 0.062 0.087" />
-                </geometry>
-        </collision>
-    </link>
-    <joint name="base_laser_vert_top_right_joint" type="fixed">
-        <parent link="base_link" />
-        <child link="laser_vert_top_right_link" />
-        <origin xyz="0.2978 -0.1450 1.8451" rpy="-1.1760 0.6313 -1.9377" />
-    </joint>
-    <link name="laser_vert_top_left_link">
-        <visual>
-                <geometry>
-                    <box size ="0.062 0.062 0.087" />
-                </geometry>
-        </visual>
-        <collision>
-                <geometry>
-                    <box size ="0.062 0.062 0.087" />
-                </geometry>
-        </collision>
-    </link>
-    <joint name="base_laser_vert_top_left_joint" type="fixed">
-        <parent link="base_link" />
-        <child link="laser_vert_top_left_link" />
-        <origin xyz="0.2997 0.1531 1.8443" rpy="1.1780 0.6198 1.9560" />
-    </joint>
-    <link name="laser_horiz_link">
-        <visual>
-                <geometry>
-                    <cylinder radius ="0.0652" length="0.072" />
-                </geometry>
-        </visual>
-        <collision>
-                <geometry>
-                    <cylinder radius ="0.0652" length="0.072" />
-                </geometry>
-        </collision>
-    </link>
-    <joint name="base_laser_horiz_joint" type="fixed">
-        <parent link="base_link" />
-        <child link="laser_horiz_link" />
-        <origin xyz="0.2325 0.0001 1.9201" rpy="-0.0012 0.1146 -0.0015" />
-    </joint>
     <xacro:macro name="xacro_name" params="side reflect">
         <link name="wheel_${side}_link">
@@ -101,5 +32,5 @@
         </link>
         <joint name="base_wheel_${side}_joint" type="continuous">
-            <parent link="base_link" />
+            <parent link="base" />
             <child link="wheel_${side}_link" />
             <origin xyz="-0.10 ${reflect * 0.4} 0.0" rpy="-1.57 0.0 0.0" />
@@ -121,5 +52,5 @@
         </link>
         <joint name="base_wheel_center_joint" type="continuous">
-            <parent link="base_link" />
+            <parent link="base" />
             <child link="wheel_center_link" />
             <origin xyz="0.10 0.0 0.0" rpy="-1.57 0.0 0.0" />
@@ -129,7 +60,11 @@
     <xacro:xacro_name side="left" reflect="1" />
     <xacro:xacro_name side="right" reflect="-1" />
-    <xacro:laser name="laser_vert_bottom" parent="base_link" xyz="0.3157894464801903 -0.002068548615034871 0.5099999434059285"
+    <xacro:laser name="laser_vert_bottom" parent="base" xyz="0.3157894464801903 -0.002068548615034871 0.5099999434059285"
             rpy="3.1354753 -1.3045001 0.0024658" meshes="package://gazebo_plugins/test/multi_robot_scenario/meshes/laser" />
-    <xacro:VLP-16 parent="base_link" name="laser_horiz" topic="laser_horiz/packets"
+    <xacro:laser name="laser_vert_top_left" parent="base" xyz="0.2997 0.1531 1.8443"
+            rpy="1.1780 0.6198 1.9560" meshes="package://gazebo_plugins/test/multi_robot_scenario/meshes/laser" />
+    <xacro:laser name="laser_vert_top_right" parent="base" xyz="0.2978 -0.1450 1.8451"
+            rpy="-1.1760 0.6313 -1.9377" meshes="package://gazebo_plugins/test/multi_robot_scenario/meshes/laser" />
+    <xacro:VLP-16 parent="base" name="laser_horiz" topic="laser_horiz/packets"
         hz="10" samples="440" gpu="false" >
         <origin xyz="0.2325416305773505 -0.0001380069427607134 1.920122926231907"
